File: can_sensor.sch (KiCad schematic (older format))
At the start: 55 parts, among them J1 TEST_1P, J2 TEST_1P, J3 TEST_1P, J4 TEST_1P, P1 SPI, P2 I2C, P4 STLink, P5 USB, P6 CAN_IN, P7 CAN_OUT, P8 TERM, Q1 Q_PMOS_GSD, SW1 RESET, SW2 BOOT, U1 NJM2870F0, U2 MIC5317, U3 STM32F042C6, U4 mcp2562

Commit message: Changed title and added pdf
Changed lines of the file:
@@
 encoding utf-8
 Sheet 1 1
-Title "Can Node"
+Title "I2C/SPI CAN Adapter"
 Date "2017-06-12"
 Rev "2.0"
@@
 On Chip Debugging connector.\nUse a stm32 Discovery board, or a STLinkv2 board.
 $Comp
-L GND #PWR028
+L GND #PWR026
 U 1 1 5880170D
 P 6825 5500
-F 0 "#PWR028" H 6825 5250 50  0001 C CNN
+F 0 "#PWR026" H 6825 5250 50  0001 C CNN
 F 1 "GND" H 6825 5350 50  0000 C CNN
 F 2 "" H 6825 5500 50  0000 C CNN
@@
 $EndComp
 $Comp
-L GND #PWR029
+L GND #PWR027
 U 1 1 59460CB0
 P 1500 2250
-F 0 "#PWR029" H 1500 2000 50  0001 C CNN
+F 0 "#PWR027" H 1500 2000 50  0001 C CNN
 F 1 "GND" H 1500 2100 50  0000 C CNN
 F 2 "" H 1500 2250 50  0001 C CNN
@@
 SPI_NSS
 $Comp
-L GND #PWR030
+L GND #PWR028
 U 1 1 57A40F91
 P 1300 4450
-F 0 "#PWR030" H 1300 4200 50  0001 C CNN
+F 0 "#PWR028" H 1300 4200 50  0001 C CNN
 F 1 "GND" H 1300 4300 50  0000 C CNN
 F 2 "" H 1300 4450 50  0000 C CNN
@@
 $EndComp
 $Comp
-L GND #PWR031
+L GND #PWR029
 U 1 1 57A40F95
 P 1300 6100
-F 0 "#PWR031" H 1300 5850 50  0001 C CNN
+F 0 "#PWR029" H 1300 5850 50  0001 C CNN
 F 1 "GND" H 1300 5950 50  0000 C CNN
 F 2 "" H 1300 6100 50  0000 C CNN
@@
 I2C_SCL
 $Comp
-L +5V #PWR032
+L +5V #PWR030
 U 1 1 59F1503E
 P 1300 3300
-F 0 "#PWR032" H 1300 3150 50  0001 C CNN
+F 0 "#PWR030" H 1300 3150 50  0001 C CNN
 F 1 "+5V" H 1300 3440 50  0000 C CNN
 F 2 "" H 1300 3300 50  0001 C CNN
@@
 $EndComp
 $Comp
-L +3.3V #PWR033
+L +3.3V #PWR031
 U 1 1 59F1527F
 P 1500 3300
-F 0 "#PWR033" H 1500 3150 50  0001 C CNN
+F 0 "#PWR031" H 1500 3150 50  0001 C CNN
 F 1 "+3.3V" H 1500 3440 50  0000 C CNN
 F 2 "" H 1500 3300 50  0001 C CNN
@@
 $EndComp
 $Comp
-L VDD #PWR034
+L VDD #PWR032
 U 1 1 59F1E45C
 P 1100 5150
-F 0 "#PWR034" H 1100 5000 50  0001 C CNN
+F 0 "#PWR032" H 1100 5000 50  0001 C CNN
 F 1 "VDD" H 1100 5300 50  0000 C CNN
 F 2 "" H 1100 5150 50  0000 C CNN
@@
 $EndComp
 $Comp
-L +5V #PWR035
+L +5V #PWR033
 U 1 1 59F1E462
 P 1300 5150
-F 0 "#PWR035" H 1300 5000 50  0001 C CNN
+F 0 "#PWR033" H 1300 5000 50  0001 C CNN
 F 1 "+5V" H 1300 5290 50  0000 C CNN
 F 2 "" H 1300 5150 50  0001 C CNN
@@
 $EndComp
 $Comp
-L +3.3V #PWR036
+L +3.3V #PWR034
 U 1 1 59F1E468
 P 1500 5150
-F 0 "#PWR036" H 1500 5000 50  0001 C CNN
+F 0 "#PWR034" H 1500 5000 50  0001 C CNN
 F 1 "+3.3V" H 1500 5290 50  0000 C CNN
 F 2 "" H 1500 5150 50  0001 C CNN
@@
 $EndComp
 Wire Wire Line
-	5100 1500 5400 1500
-Wire Wire Line
-	5400 1500 5700 1500
-Wire Wire Line
-	4050 1500 4050 1700
-Wire Wire Line
-	4050 1700 4050 1900
+	5100 1500 5700 1500
+Wire Wire Line
+	4050 1500 4050 1900
 Wire Wire Line
 	3200 1500 3500 1500
 Wire Wire Line
-	3800 1500 4050 1500
-Wire Wire Line
-	4050 1500 4100 1500
-Wire Wire Line
-	3800 2200 4050 2200
-Wire Wire Line
-	4050 2200 4600 2200
-Wire Wire Line
-	4600 2200 5100 2200
-Wire Wire Line
-	5100 2200 5400 2200
-Wire Wire Line
-	5400 2200 5700 2200
-Wire Wire Line
-	4600 2150 4600 2200
-Wire Wire Line
-	4600 2200 4600 2300
+	3800 1500 4100 1500
+Wire Wire Line
+	3800 2200 5700 2200
+Wire Wire Line
+	4600 2150 4600 2300
 Wire Wire Line
 	4050 2200 4050 2100
@@
 Connection ~ 4050 1500
 Wire Wire Line
-	5000 2750 5000 2800
-Wire Wire Line
-	5000 2800 5000 2950
-Wire Wire Line
-	4850 2800 5000 2800
-Wire Wire Line
-	5000 2800 5150 2800
-Wire Wire Line
-	5150 2800 5300 2800
-Wire Wire Line
-	5300 2800 5450 2800
+	5000 2750 5000 2950
+Wire Wire Line
+	4850 2800 5450 2800
 Connection ~ 5400 1500
 Connection ~ 5000 2800
@@
 Connection ~ 3500 1500
 Wire Wire Line
-	2700 2150 2700 2200
-Wire Wire Line
-	2700 2200 2700 2300
-Wire Wire Line
-	1000 2200 1500 2200
-Wire Wire Line
-	1500 2200 1800 2200
-Wire Wire Line
-	1800 2200 2700 2200
-Wire Wire Line
-	2700 2200 3200 2200
-Wire Wire Line
-	3200 2200 3500 2200
-Wire Wire Line
-	1200 1500 1500 1500
-Wire Wire Line
-	1500 1500 1800 1500
-Wire Wire Line
-	1800 1500 2200 1500
+	2700 2150 2700 2300
+Wire Wire Line
+	1000 2200 3500 2200
+Wire Wire Line
+	1200 1500 2200 1500
 Wire Wire Line
 	1800 2100 1800 2200
@@
 Connection ~ 1800 1500
 Wire Wire Line
-	1500 1400 1500 1500
-Wire Wire Line
-	1500 1500 1500 1900
-Wire Wire Line
-	1500 2100 1500 2200
-Wire Wire Line
-	1500 2200 1500 2250
+	1500 1400 1500 1900
+Wire Wire Line
+	1500 2100 1500 2250
 Connection ~ 1800 2200
 Wire Wire Line
-	3800 1400 3800 1500
-Wire Wire Line
-	3800 1500 3800 1900
+	3800 1400 3800 1900
 Wire Wire Line
 	3800 2100 3800 2200
@@
 Connection ~ 3800 1500
 Wire Wire Line
-	1800 1500 1800 1700
-Wire Wire Line
-	1800 1700 1800 1900
+	1800 1500 1800 1900
 Connection ~ 1500 1500
 Wire Wire Line
@@
 	8600 1600 8600 1700
 Wire Wire Line
-	8600 2000 8600 2050
-Wire Wire Line
-	8600 2050 8600 2100
+	8600 2000 8600 2100
 Wire Wire Line
 	8975 3500 9075 3500
 Wire Wire Line
-	9075 3500 9075 3800
-Wire Wire Line
-	9075 3800 9075 3900
+	9075 3500 9075 3900
 Wire Wire Line
 	9075 3800 8975 3800
@@
 	1450 6800 1400 6800
 Wire Wire Line
-	1400 7200 1400 7400
-Wire Wire Line
-	1400 7400 1400 7500
-Wire Wire Line
-	1000 7400 1400 7400
-Wire Wire Line
-	1400 7400 1600 7400
+	1400 7200 1400 7500
+Wire Wire Line
+	1000 7400 1600 7400
 Connection ~ 1400 7400
 Wire Wire Line
@@
 Connection ~ 5150 6450
 Wire Wire Line
-	3500 1400 3500 1500
-Wire Wire Line
-	3500 1500 3500 1900
+	3500 1400 3500 1900
 Wire Wire Line
 	3500 2200 3500 2100
@@
 Connection ~ 1800 1700
 Wire Wire Line
-	5700 1400 5700 1500
-Wire Wire Line
-	5700 1500 5700 1900
+	5700 1400 5700 1900
 Wire Wire Line
 	5700 2200 5700 2100
@@
 	7650 2650 7650 2700
 Wire Wire Line
-	4900 6450 5150 6450
-Wire Wire Line
-	5150 6450 5450 6450
+	4900 6450 5450 6450
 Wire Wire Line
 	7850 2650 7850 2700
@@
 	4000 2950 4000 2800
 Wire Wire Line
-	4000 2800 4250 2800
-Wire Wire Line
-	4250 2800 4400 2800
-Wire Wire Line
-	4400 2800 4550 2800
-Wire Wire Line
-	4550 2800 4700 2800
+	4000 2800 4700 2800
 Wire Wire Line
 	4250 2800 4250 2950
@@
 	5350 6950 5350 6650
 Wire Wire Line
-	4900 6950 5150 6950
-Wire Wire Line
-	5150 6950 5350 6950
+	4900 6950 5350 6950
 Connection ~ 5150 6950
 Wire Wire Line
@@
 	6200 4450 6250 4450
 Wire Wire Line
-	1200 5950 1300 5950
-Wire Wire Line
-	1300 5950 2000 5950
-Wire Wire Line
-	1200 4300 1300 4300
-Wire Wire Line
-	1300 4300 2150 4300
+	1200 5950 2000 5950
+Wire Wire Line
+	1200 4300 2150 4300
 Wire Wire Line
 	1300 4300 1300 4450
@@
 	6150 2700 6150 2650
 Wire Wire Line
-	6150 2650 6350 2650
-Wire Wire Line
-	6350 2650 6650 2650
-Wire Wire Line
-	6650 2650 6850 2650
-Wire Wire Line
-	6850 2650 7000 2650
-Wire Wire Line
-	7000 2650 7150 2650
-Wire Wire Line
-	7150 2650 7350 2650
-Wire Wire Line
-	7350 2650 7650 2650
-Wire Wire Line
-	7650 2650 7850 2650
+	6150 2650 7850 2650
 Wire Wire Line
 	6350 2700 6350 2650
@@
 	7850 2950 7850 2900
 Wire Wire Line
-	6150 2950 6350 2950
-Wire Wire Line
-	6350 2950 6650 2950
-Wire Wire Line
-	6650 2950 6850 2950
-Wire Wire Line
-	6850 2950 7000 2950
-Wire Wire Line
-	7000 2950 7150 2950
-Wire Wire Line
-	7150 2950 7350 2950
-Wire Wire Line
-	7350 2950 7650 2950
-Wire Wire Line
-	7650 2950 7850 2950
+	6150 2950 7850 2950
 Wire Wire Line
 	6150 2950 6150 2900
@@
 	5900 6850 5900 6950
 Wire Wire Line
-	5900 6400 5900 6500
-Wire Wire Line
-	5900 6500 5900 6550
+	5900 6400 5900 6550
 Wire Wire Line
 	6100 6200 6100 6125
@@
 	1000 1800 1000 2200
 Wire Wire Line
-	8600 2200 8600 2250
-Wire Wire Line
-	8600 2250 8600 2350
+	8600 2200 8600 2350
 Wire Wire Line
 	8700 2050 8600 2050
@@
 	2575 4900 3500 4900
 Wire Wire Line
-	1300 3550 1300 3650
-Wire Wire Line
-	1300 3650 1300 3800
+	1300 3550 1300 3800
 Wire Wire Line
 	1300 3800 1200 3800
@@
 	1500 3650 1500 3550
 Wire Wire Line
-	1100 3650 1300 3650
-Wire Wire Line
-	1300 3650 1500 3650
-Wire Wire Line
-	1500 3650 2150 3650
+	1100 3650 2150 3650
 Connection ~ 1300 3650
 Wire Wire Line
 	1100 3550 1100 3650
 Wire Wire Line
-	1500 3300 1500 3325
-Wire Wire Line
-	1500 3325 1500 3350
+	1500 3300 1500 3350
 Wire Wire Line
 	1300 3300 1300 3350
@@
 Connection ~ 1500 3325
 Wire Wire Line
-	1300 5400 1300 5500
-Wire Wire Line
-	1300 5500 1300 5650
+	1300 5400 1300 5650
 Wire Wire Line
 	1500 5500 1500 5400
 Wire Wire Line
-	1100 5500 1300 5500
-Wire Wire Line
-	1300 5500 1500 5500
-Wire Wire Line
-	1500 5500 2000 5500
+	1100 5500 2000 5500
 Connection ~ 1300 5500
 Wire Wire Line
@@
 	1500 5150 1500 5200
 Wire Wire Line
-	2575 4275 2725 4275
-Wire Wire Line
-	2725 4275 2825 4275
-$Comp
-L +3.3V #PWR037
+	2575 4275 2825 4275
+$Comp
+L +3.3V #PWR035
 U 1 1 59F2B384
 P 2725 4250
-F 0 "#PWR037" H 2725 4100 50  0001 C CNN
+F 0 "#PWR035" H 2725 4100 50  0001 C CNN
 F 1 "+3.3V" H 2725 4390 50  0000 C CNN
 F 2 "" H 2725 4250 50  0001 C CNN
